Commit message: hooly

File: install/linorobot2_description/share/linorobot2_description/urdf/mecanum_properties.urdf.xacro (robot description, xacro)
@@ -15,9 +15,3 @@
     <origin xyz="-0.0475 0 0.125" rpy="0 0 0"/>
   </xacro:property>
-  <xacro:property name="depth_sensor_pose">
-    <origin xyz="0.2375 0 0.06" rpy="0 0 0"/>
-  </xacro:property>
-  <xacro:property name="sonar_pose">
-    <origin xyz="0.22 0 0" rpy="0 0 0"/>
-  </xacro:property>
 </robot>

File: install/linorobot2_description/share/linorobot2_description/urdf/robots/mecanum.urdf.xacro (robot description, xacro)
@@ -57,10 +57,4 @@
     <xacro:insert_block name="laser_pose" />
   </xacro:generic_laser>
-  <xacro:depth_sensor>
-    <xacro:insert_block name="depth_sensor_pose" />
-  </xacro:depth_sensor>
-  <xacro:sonar>
-    <xacro:insert_block name="sonar_pose" />
-  </xacro:sonar>
   <xacro:omni_drive_controller/>
 </robot>
